File: Hardware/Brady_Davis/Brady_Davis.kicad_sch (KiCad schematic)
At the start: 10 parts, among them J1 RJ45_LED_Shielded, J2 Conn_02x03_Counter_Clockwise, Q1 Q_PMOS_GDS, Q2 Q_NMOS_GSD, U1 Teensy4.1_DEV-16771

Commit message: Layout Training
Parts:
- added C2, C3: 10uF, Capacitor_SMD:C_0603_1608Metric_Pad1.08x0.95mm_HandSolder, symbol Device:C
- added U2: OKI-78SR-3.3_1.5-W36H-C, Converter_DCDC:Converter_DCDC_Murata_OKI-78SR_Horizontal, symbol Converter_DCDC:OKI-78SR-3.3_1.5-W36H-C
- C1: footprint (none) -> Capacitor_SMD:C_0603_1608Metric_Pad1.08x0.95mm_HandSolder
- Conn1, Conn2: footprint (none) -> MRDT_Connectors:Square_Anderson_2_H_Side_By_Side
- J1: footprint (none) -> MRDT_Connectors:RJ45_Teensy
- J2: footprint (none) -> Connector_PinHeader_2.00mm:PinHeader_2x03_P2.00mm_Vertical
- Q1: footprint (none) -> Package_TO_SOT_SMD:TO-252-2
- Q2: footprint (none) -> Package_TO_SOT_SMD:SOT-23
- R1, R2: footprint (none) -> Resistor_SMD:R_0603_1608Metric_Pad0.98x0.95mm_HandSolder
- U1: footprint MODULE_DEV-16771 -> MRDT_Shields:Teensy_4_1_Vertical
Connections:
- net +36V: now also C2.1, U2.1 (IN)
- net +3V3: now also C3.1, U2.3 (OUT)
- net GND: now also C2.2, C3.2, U2.2 (GND)
- net at Q1.2 (D): now also Conn2.2 (V+Log); no longer Conn2.1
- net Tx+: now reaches J1.1, J2.1 (Pin_1)
- net Tx-: now reaches J1.3, J2.2 (Pin_2)
- net Rx+: now reaches J1.4, J2.6 (Pin_6)
- net Rx-: now reaches J1.6, J2.5 (Pin_5)
