File: Hardware/Brady_Davis/Brady_Davis.kicad_sch (KiCad schematic)
At the start: 13 parts, among them J1 RJ45_LED_Shielded, J2 Conn_02x03_Counter_Clockwise, Q1 Q_PMOS_GDS, Q2 Q_NMOS_GSD, U1 Teensy4.1_DEV-16771, U2 OKI

Commit message: layout shtuff
Other:
- note added: "OKI"
Changed lines of the file:
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@@
+    (stroke (width 0) (type default) (color 0 0 0 0))
+  )
+  (polyline (pts (xy 150.495 139.065) (xy 228.6 139.065))
     (stroke (width 0) (type default) (color 0 0 0 0))
   )
   (wire (pts (xy 204.47 40.64) (xy 209.55 40.64))
+    (stroke (width 0) (type default) (color 0 0 0 0))
+  )
+  (polyline (pts (xy 228.6 139.065) (xy 228.6 70.485))
     (stroke (width 0) (type default) (color 0 0 0 0))
   )
@@
     (effects (font (size 5 5)) (justify left bottom))
   )
+  (text "OKI" (at 189.23 121.285 0)
+    (effects (font (size 2.54 2.54)) (justify left bottom))
+  )
   (text "Brady_Davis Rev1" (at 483.235 401.32 0)
