File: Hardware/Ethan_Medrow/Ethan_Medrow.kicad_sch (KiCad schematic)
At the start: 10 parts, among them J1 Conn_02x03_Counter_Clockwise, J2 RJ45_LED_Shielded, Q1 Q_PMOS_GDS, Q2 Q_NMOS_GSD, U1 Teensy4.1_DEV-16771

Commit message: Made Layout
Added Footprints. Made Layout.
Parts:
- added C2, C3: 10uF, Capacitor_SMD:C_0603_1608Metric_Pad1.08x0.95mm_HandSolder, symbol Device:C
- added U2: OKI, MRDT_Devices:OKI_Horizontal, symbol MRDT_Devices:OKI
- C1: footprint (none) -> Capacitor_SMD:C_0603_1608Metric_Pad1.08x0.95mm_HandSolder
- Conn1, Conn2: footprint (none) -> MRDT_Connectors:Square_Anderson_2_H_Side_By_Side_PV
- J1: footprint (none) -> Connector_PinHeader_2.00mm:PinHeader_2x03_P2.00mm_Vertical
- J2: footprint (none) -> MRDT_Connectors:RJ45_Teensy
- Q1: footprint (none) -> Package_TO_SOT_SMD:TO-252-2
- Q2: footprint (none) -> Package_TO_SOT_SMD:SOT-23
- R1, R2: footprint (none) -> Resistor_SMD:R_0603_1608Metric_Pad0.98x0.95mm_HandSolder
- U1: footprint MODULE_DEV-16771 -> MRDT_Shields:Teensy_4_1_Vertical
Connections:
- net +36V: now also C2.1, U2.1 (Vi)
- net +3V3: now also C3.1, U2.3 (Vo)
- net GND: now also C2.2, C3.2, U2.2 (GND)
- net at Q1.2 (D): now also Conn2.4 (PV+); no longer Conn2.1
- net Tx +: now reaches J1.1 (Pin_1), J2.1
- net Rx -: now reaches C1.1, J1.5 (Pin_5), J2.2, J2.5, J2.6
- net Tx -: now reaches J1.2 (Pin_2), J2.3
- net Rx +: now reaches J1.6 (Pin_6), J2.4
- net at C1.2, J2.8, J2.9: now also J1.3 (Pin_3)
Other:
- note added: "Oki"
